File: jlcpcb-vertical/usb_c_cable_tester.kicad_sch (KiCad schematic)
At the start: 58 parts, among them J1 USB C, J2 USB C, J3 USB_B_Micro, J4 USB3_B, J5 USB_B_Mini, J6 USB3_A

Commit message: jlcpcb-vertical/ v3.0b. Spacing, MicroB with long pins, added battery test.
Parts:
- added D26: LED, LED_SMD:LED_0603_1608Metric_Pad1.05x0.95mm_HandSolder, symbol Device:LED_Small_Filled
- added R26: 2.2k, Resistor_SMD:R_0603_1608Metric_Pad0.98x0.95mm_HandSolder, symbol Device:R_Small
- added SW1: Battery, Button_Switch_SMD:SW_SPST_TS-1088-xR020, symbol Switch:SW_Push
- BT1: footprint easyeda:BAT-TH_CR2032-BS-6-1 -> Battery:BatteryHolder_Keystone_1060_1x2032
- J3: Alt LCSC C668588 -> C145795; LCSC C456007 -> C145794
Connections:
- net +3V3: now also SW1.1
- net GND: now also D26.1 (K)
- new net: D26.2 (A), R26.2
- new net: R26.1, SW1.2
